File: bms_segment.kicad_pcb (KiCad board)
At the start: 4 copper layers, 70 x 100 mm, 219 parts, among them J1 Conn_02x09_Counter_Clockwise, J2 Conn_02x09_Counter_Clockwise, J3 Conn_02x10_Odd_Even, J4 Conn_02x10_Odd_Even, J5 Conn_01x04, J6 Conn_01x04, J7 Conn_01x06, Q1 IRLML0060, Q10 IRLML0060, Q11 IRLML0060, Q12 IRLML0060, Q13 IRLML0060, Q14 IRLML0060, Q15 IRLML0060, Q16 IRLML0060, Q17 BSS84, Q2 IRLML0060, Q3 IRLML0060, Q4 IRLML0060, Q5 IRLML0060, Q6 IRLML0060, Q7 IRLML0060, Q8 IRLML0060, Q9 IRLML0060, SW1 SW_Push, U1 LMR516xx, U2 MAX14921, U3 MAX11163, U4 REF61xx, U5 STM32F103C8Tx, U6 ADuM1252, U7 74LV4051A, U8 74LV4051A, U9 74LV4051A

Commit message: Revision E
Parts:
- removed the H4 at (164.0, 139.5)
- removed J1, J2: Conn_02x09_Counter_Clockwise, yfs:MolexMilliGrid2x9
- removed R10, R11, R12, R13, R14, R15, R16, R17, R18, R19, R20, R21, R22, R27, R30, R33, R36, R39, R42, R45, R48, R51, R54, R57, R60, R63, R66, R69, R7, R72, R8, R9: 3k, Resistor_SMD:R_0603_1608Metric
- removed kibuzzard-69C6C1F9: G***, kibuzzard-69C6C1F9
- added G***: LOGO, LOGO, B.Cu at (192.8, 88.1)
- added G****: LOGO, LOGO, F.Cu at (159.5, 62.0)
- added H4: MountingHole, MountingHole:MountingHole_3.2mm_M3, F.Cu at (182.2, 62.0)
- added H4: MountingHole, MountingHole:MountingHole_3.2mm_M3, F.Cu at (205.5, 54.5)
- added H4: MountingHole, MountingHole:MountingHole_3.2mm_M3, F.Cu at (215.0, 107.5)
- added H4: MountingHole, MountingHole:MountingHole_3.2mm_M3, F.Cu at (182.5, 54.5)
- added H4: MountingHole, MountingHole:MountingHole_3.2mm_M3, F.Cu at (206.2, 62.0)
- added H4: MountingHole, MountingHole:MountingHole_3.2mm_M3, F.Cu at (182.5, 112.5)
- added H4: MountingHole, MountingHole:MountingHole_3.2mm_M3, F.Cu at (206.2, 105.0)
- added H4: MountingHole, MountingHole:MountingHole_3.2mm_M3, F.Cu at (205.5, 112.5)
- added HS1: Heatsink, TestPoint:TestPoint_Pad_D1.0mm, F.Cu at (219.5, 52.0)
- added HS2: PLACEHOLDER, TestPoint:TestPoint_Pad_D1.0mm, F.Cu at (356.5, 61.5)
- added J10: Conn_02x17_Counter_Clockwise, yfs:SAMTEC_TW-17-03-F-D-275-090, F.Cu at (205.2, 67.5)
- added RN13: 3k, Resistor_SMD:R_Array_Concave_4x0603, F.Cu at (174.0, 110.8)
- added RN14: 3k, Resistor_SMD:R_Array_Concave_4x0603, F.Cu at (174.0, 104.2)
- added RN15: 3k, Resistor_SMD:R_Array_Concave_4x0603, F.Cu at (174.0, 97.8)
- added RN16: 3k, Resistor_SMD:R_Array_Concave_4x0603, F.Cu at (174.0, 91.2)
- added RN17: 3k, Resistor_SMD:R_Array_Concave_4x0603, F.Cu at (174.0, 84.8)
- added RN18: 3k, Resistor_SMD:R_Array_Concave_4x0603, F.Cu at (174.0, 78.2)
- added RN19: 3k, Resistor_SMD:R_Array_Concave_4x0603, F.Cu at (174.0, 71.8)
- added RN20: 3k, Resistor_SMD:R_Array_Concave_4x0603, F.Cu at (174.0, 65.5)
- added kibuzzard-69D1B272: G***, kibuzzard-69D1B272, F.Cu at (211.7, 104.2)
- added kibuzzard-69D2F3F3: G***, kibuzzard-69D2F3F3, F.Cu at (211.7, 62.8)
- J5, J6: footprint Connector_JST:JST_PH_B4B-PH-K_1x04_P2.00mm_Vertical -> yfs:MolexMicrofitPlus2x2-RA
- JP1, JP2, JP3, JP4, RN10, RN12, RN4, RN6, RN8: moved to B.Cu
- moved TH2 150.2 mm to (192.0, 79.2), turned to 90 degrees
- moved TH3 146.9 mm to (192.0, 92.2), turned to 90 degrees
- moved TH4 144.2 mm to (192.0, 105.3), turned to 90 degrees
- moved RN1 132.0 mm to (170.0, 54.8)
- moved C36 118.6 mm to (145.6, 54.6), turned to -45 degrees
- moved D17 117.7 mm to (152.0, 55.5), turned to 180 degrees
- moved C38 116.8 mm to (140.5, 54.5), turned to -135 degrees
- moved C35 116.5 mm to (149.8, 63.8), turned to -135 degrees
- moved D1 114.8 mm to (215.0, 64.8), turned to 180 degrees
- moved J7 113.6 mm to (161.5, 53.7), turned to 180 degrees
- moved C37 112.0 mm to (138.0, 57.0), turned to 45 degrees
- moved Q1 111.9 mm to (190.8, 54.0), turned to 180 degrees
- moved R28 111.9 mm to (197.2, 54.0)
- moved D2 110.8 mm to (215.0, 67.2), turned to 180 degrees
- moved C10 109.5 mm to (148.2, 77.8), turned to 180 degrees
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Connections:
- C12 pad 1: Net-(U2-CB16) -> Net-(U2-CT16)
- C12 pad 2: Net-(U2-CT16) -> Net-(U2-CB16)
- Q1 pad 1: Net-(Q1-G) -> /Balancers/BA1
- Q10 pad 1: Net-(Q10-G) -> /Balancers/BA10
- Q11 pad 1: Net-(Q11-G) -> /Balancers/BA11
- Q12 pad 1: Net-(Q12-G) -> /Balancers/BA12
- Q13 pad 1: Net-(Q13-G) -> /Balancers/BA13
- Q14 pad 1: Net-(Q14-G) -> /Balancers/BA14
- Q15 pad 1: Net-(Q15-G) -> /Balancers/BA15
- Q16 pad 1: Net-(Q16-G) -> /Balancers/BA16
- Q2 pad 1: Net-(Q2-G) -> /Balancers/BA2
- Q3 pad 1: Net-(Q3-G) -> /Balancers/BA3
- Q4 pad 1: Net-(Q4-G) -> /Balancers/BA4
- Q5 pad 1: Net-(Q5-G) -> /Balancers/BA5
- Q6 pad 1: Net-(Q6-G) -> /Balancers/BA6
- Q7 pad 1: Net-(Q7-G) -> /Balancers/BA7
- Q8 pad 1: Net-(Q8-G) -> /Balancers/BA8
- Q9 pad 1: Net-(Q9-G) -> /Balancers/BA9
- U2 pad 15: Net-(U2-CV16) -> CV16
- U2 pad 16: /Balancers/BA16 -> BA16
- U2 pad 19: Net-(U2-CV15) -> CV15
- U2 pad 20: /Balancers/BA15 -> BA15
- U2 pad 23: Net-(U2-CV14) -> CV14
- U2 pad 24: /Balancers/BA14 -> BA14
- U2 pad 27: Net-(U2-CV13) -> CV13
- U2 pad 28: /Balancers/BA13 -> BA13
- U2 pad 31: Net-(U2-CV12) -> CV12
- U2 pad 32: /Balancers/BA12 -> BA12
- U2 pad 35: Net-(U2-CV11) -> CV11
- U2 pad 36: /Balancers/BA11 -> BA11
- U2 pad 39: Net-(U2-CV10) -> CV10
- U2 pad 40: /Balancers/BA10 -> BA10
- U2 pad 43: Net-(U2-CV9) -> CV9
- U2 pad 44: /Balancers/BA9 -> BA9
- U2 pad 47: Net-(U2-CV8) -> CV8
- U2 pad 48: /Balancers/BA8 -> BA8
- U2 pad 51: Net-(U2-CV7) -> CV7
- U2 pad 52: /Balancers/BA7 -> BA7
- U2 pad 55: Net-(U2-CV6) -> CV6
- U2 pad 56: /Balancers/BA6 -> BA6
- U2 pad 59: Net-(U2-CV5) -> CV5
- U2 pad 60: /Balancers/BA5 -> BA5
- U2 pad 63: Net-(U2-CV4) -> CV4
- U2 pad 64: /Balancers/BA4 -> BA4
- U2 pad 67: Net-(U2-CV3) -> CV3
- U2 pad 68: /Balancers/BA3 -> BA3
- U2 pad 71: Net-(U2-CV2) -> CV2
- U2 pad 72: /Balancers/BA2 -> BA2
- U2 pad 75: Net-(U2-CV1) -> CV1
- U2 pad 76: /Balancers/BA1 -> BA1
- U7 pad 1: /Thermistor Sampling/Thermistors/TH5 -> /Thermistor Sampling/Thermistors/TH7
- U7 pad 13: /Thermistor Sampling/Thermistors/TH1 -> /Thermistor Sampling/Thermistors/TH3
- U7 pad 15: /Thermistor Sampling/Thermistors/TH3 -> /Thermistor Sampling/Thermistors/TH1
- U7 pad 2: /Thermistor Sampling/Thermistors/TH7 -> /Thermistor Sampling/Thermistors/TH8
- U7 pad 4: /Thermistor Sampling/Thermistors/TH8 -> /Thermistor Sampling/Thermistors/TH5
- U8 pad 1: /Thermistor Sampling/Thermistors/TH13 -> /Thermistor Sampling/Thermistors/TH12
- U8 pad 12: /Thermistor Sampling/Thermistors/TH12 -> /Thermistor Sampling/Thermistors/TH13
- U8 pad 13: /Thermistor Sampling/Thermistors/TH9 -> /Thermistor Sampling/Thermistors/TH14
- U8 pad 14: /Thermistor Sampling/Thermistors/TH10 -> /Thermistor Sampling/Thermistors/TH16
- U8 pad 4: /Thermistor Sampling/Thermistors/TH16 -> /Thermistor Sampling/Thermistors/TH9
- U8 pad 5: /Thermistor Sampling/Thermistors/TH14 -> /Thermistor Sampling/Thermistors/TH10
- U9 pad 1: /Thermistor Sampling/Thermistors/TH21 -> /Thermistor Sampling/Thermistors/TH19
- U9 pad 12: /Thermistor Sampling/Thermistors/TH20 -> /Thermistor Sampling/Thermistors/TH21
- U9 pad 13: /Thermistor Sampling/Thermistors/TH17 -> /Thermistor Sampling/Thermistors/TH22
- U9 pad 14: /Thermistor Sampling/Thermistors/TH18 -> /Thermistor Sampling/Thermistors/TH23
- U9 pad 15: /Thermistor Sampling/Thermistors/TH19 -> /Thermistor Sampling/Thermistors/TH24
- U9 pad 2: /Thermistor Sampling/Thermistors/TH23 -> /Thermistor Sampling/Thermistors/TH20
- U9 pad 4: /Thermistor Sampling/Thermistors/TH24 -> /Thermistor Sampling/Thermistors/TH18
- U9 pad 5: /Thermistor Sampling/Thermistors/TH22 -> /Thermistor Sampling/Thermistors/TH17
Routing:
- net /Thermistor Sampling/Thermistors/PWR: track 0.00 -> 251.3 mm, vias 0 -> 5
- net TAP16: track 6.67 -> 96.2 mm, vias 0 -> 1
- net +3V3: track 25.6 -> 98.8 mm, vias 14 -> 63
- net /SCL: track 0.00 -> 68.9 mm, vias 0 -> 3
- net /Thermistor Sampling/Thermistors/Network1/IN_2: track 0.00 -> 66.8 mm, vias 0 -> 2
- net /SDA: track 0.00 -> 64.2 mm, vias 0 -> 3
- net TAP14: track 11.9 -> 73.9 mm, vias 0 -> 1
- net /Thermistor Sampling/Thermistors/TH3: track 0.00 -> 61.5 mm, vias 0 -> 2
- net /Thermistor Sampling/EN: track 0.00 -> 60.2 mm, vias 0 -> 5
- net /Thermistor Sampling/Thermistors/TH4: track 0.00 -> 59.8 mm, vias 0 -> 2
- net TAP1: track 11.9 -> 71.2 mm, vias 0 -> 1
- net TAP12: track 11.9 -> 71.0 mm, vias 0 -> 1
- net TAP4: track 11.9 -> 69.1 mm, vias 0 -> 1
- net TAP10: track 11.9 -> 68.0 mm, vias 0 -> 1
- net /Thermistor Sampling/Thermistors/Network1/IN_1: track 0.00 -> 55.5 mm, vias 0 -> 2
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- added copper zone on In2.Cu, net +3V3
- added copper zone on In2.Cu, net +5VA
- added copper zone on B.Cu, net GND
- added copper zone on F.Cu, net GND
- added copper zone on In1.Cu, net GND
- added copper zone on In2.Cu, net GND
Other:
- board size 70 x 100 mm -> 120 x 65 mm
- board text added: "${PCB_DATE}"
- board text added: "2.0mm"
- board text added: "3V3"
- board text added: "ADR[3:0]"
- board text added: "AOUT"
- board text added: "BMS"
- board text added: "BY LOGAN C + OWEN S"
- board text added: "C1"
- board text added: "C10"
- board text added: "C11"
- board text added: "C12"
- board text added: "C13"
- board text added: "C14"
- board text added: "C15"
- board text added: "C16"
- board text added: "C2"
- board text added: "C3"
- board text added: "C4"
- board text added: "C5"
- board text added: "C6"
- board text added: "C7"
- board text added: "C8"
- board text added: "C9"
- board text added: "DISTRIBUTED BMS"
- board text added: "GND"
- board text added: "HOT SURFACE"
- board text added: "I2C"
- board text added: "REF"
- board text added: "REV ${REVISION}"
- board text added: "RST"
- board text added: "SW"
- board text added: "SWD"
- board text added: "VIN"
- board text added: "york-fs/bms-segment"
