File: daughter-14s/daughter_14s.kicad_pcb (KiCad board)
At the start: 4 copper layers, 34 x 50 mm, 37 parts, among them J1 Conn_02x08_Counter_Clockwise, J10 Conn_02x17_Counter_Clockwise

Commit message: daughter-14s: Cleanup
Parts:
- TP1: footprint yfs:KEYSTONE_5019 -> TestPoint:TestPoint_Keystone_5019_Miniature
- renumbered J10 to J1, J1 to J2

Commit message: daughter-14s: Disable inner layers
Routing:
- net TAP14: track 26.5 -> 26.0 mm
Other:
- copper layers 4 -> 2
Changed lines of the file:
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@@
 	(layers
 		(0 "F.Cu" signal)
-		(4 "In1.Cu" signal)
-		(6 "In2.Cu" signal)
 		(2 "B.Cu" signal)
 		(5 "F.SilkS" user "F.Silkscreen")
@@
 			)
 			(layer "dielectric 1"
-				(type "prepreg")
-				(thickness 0.2104)
-				(material "FR4")
-				(epsilon_r 4.4)
-				(loss_tangent 0.02)
-			)
-			(layer "In1.Cu"
-				(type "copper")
-				(thickness 0.0152)
-			)
-			(layer "dielectric 2"
 				(type "core")
-				(thickness 1.065)
-				(material "FR4")
-				(epsilon_r 4.6)
-				(loss_tangent 0.02)
-			)
-			(layer "In2.Cu"
-				(type "copper")
-				(thickness 0.0152)
-			)
-			(layer "dielectric 3"
-				(type "prepreg")
-				(thickness 0.2104)
+				(thickness 1.5162)
 				(material "FR4")
 				(epsilon_r 4.4)
@@
 	)
 	(segment
-		(start 205.25 69.500001)
-		(end 205.250001 69.5)
-		(width 0.5)
-		(layer "In2.Cu")
-		(net 3)
-	)
-	(segment
 		(start 193.9 72)
 		(end 201.25 72)
@@
 	)
 	(segment
-		(start 204.9125 73.2)
-		(end 205.25 73.5375)
-		(width 0.2)
-		(layer "In2.Cu")
-		(net 12)
-	)
-	(segment
 		(start 193.9 77)
 		(end 201.25 77)
@@
 	)
 	(segment
-		(start 204.8875 95.9)
-		(end 205.25 95.5375)
-		(width 0.2)
-		(layer "In2.Cu")
-		(net 15)
-	)
-	(segment
 		(start 184.75 67.5)
 		(end 187.75 64.5)
@@
 		(net 0)
 		(net_name "")
-		(layers "F.Cu" "B.Cu" "In1.Cu" "In2.Cu")
+		(layers "F.Cu" "B.Cu")
 		(hatch edge 0.5)
 		(connect_pads
